Commit message: change file position

File: catkin_ws/src/choreonoid_ros_control_assembler_sample/urdf/one_joint_robot.xacro (robot description, xacro)
@@ -1,17 +1,5 @@
 <?xml version="1.0" ?>
 <robot name="test_robot" xmlns:xacro="http://ros.org/wiki/xacro">
-  <!-- copy from cnoid_tank_pkgs/cnoid_tank_description/urdf/common.xacro -->
-  <xacro:property name="M_PI" value="3.14159274"/>
-  <xacro:macro name="joint_position_trans_v0" params="name">
-	<transmission name="${name}_trans">
-      <type>transmission_interface/SimpleTransmission</type>
-      <joint name="${name}">
-		<hardwareInterface>PositionJointInterface</hardwareInterface>
-      </joint>
-	  <actuator name="${name}_motor">
-		<hardwareInterface>PositionJointInterface</hardwareInterface>
-      </actuator>
-	</transmission>
-  </xacro:macro>
+  <xacro:include filename="$(find choreonoid_ros_control_assembler_sample)/urdf/common.xacro"/>
   <link name="Root">
     <visual>
