Commit message: change position paramter

File: catkin_ws/src/choreonoid_ros_control_assembler_sample/urdf/two_joint_robot.xacro (robot description, xacro)
@@ -9,5 +9,5 @@
     <parent link="Root"/>
     <child link="LINK_0"/>
-    <origin xyz="0.000000 0.000000 0.000000" rpy="0 0 0" />
+    <origin xyz="0.000000 0.000000 0.019000" rpy="0 0 0" />
     <axis xyz="0.000000 0.000000 1.000000"/>
     <limit lower="-3.141593" upper="3.141593" velocity="5" effort="500"/>
@@ -18,5 +18,5 @@
     <parent link="LINK_0"/>
     <child link="FR12_H101_S_28_2"/>
-    <origin xyz="0.000000 0.000000 0.000000" rpy="0 0 0" />
+    <origin xyz="0.008000 0.059200 -0.007000" rpy="0 0 0" />
   </joint>
   <link name="LINK_1">
@@ -25,5 +25,5 @@
     <parent link="FR12_H101_S_28_2"/>
     <child link="LINK_1"/>
-    <origin xyz="0.000000 0.000000 0.000000" rpy="0 0 0" />
+    <origin xyz="0.007000 -0.008000 0.032700" rpy="0 0 0" />
     <axis xyz="-0.000000 -0.000000 -1.000000"/>
     <limit lower="-3.141593" upper="3.141593" velocity="5" effort="500"/>
